File: Hardware/Geiger Counter Mainboard/KiCad/Geiger Counter Mainboard.kicad_pcb (KiCad board)
At the start: 2 copper layers, 0 parts

Commit message: Added PCB for mainboard
Parts:
- added BZ1: Buzzer, Connector_PinHeader_2.54mm:PinHeader_1x02_P2.54mm_Vertical, F.Cu at (132.8, 142.4)
- added C1: 10nF, Capacitor_SMD:C_1206_3216Metric_Pad1.33x1.80mm_HandSolder, F.Cu at (153.4, 140.8)
- added C2: 100uF, Capacitor_SMD:CP_Elec_6.3x5.4, F.Cu at (160.8, 143.1)
- added D1: 1N4148WS, Diode_SMD:D_SOD-323_HandSoldering, F.Cu at (131.6, 139.1)
- added H1: MountingHole_Pad, Footprints:MountingHole_3.2mm_M3_Pad_Via, F.Cu at (107.9, 144.0)
- added H2: MountingHole_Pad, Footprints:MountingHole_3.2mm_M3_Pad_Via, F.Cu at (191.2, 144.0)
- added J1: FOLLOWER TUBE(S), Connector_PinHeader_2.54mm:PinHeader_1x03_P2.54mm_Vertical, F.Cu at (183.6, 145.9)
- added J2: MAIN TUBE(S), Connector_PinHeader_2.54mm:PinHeader_1x03_P2.54mm_Vertical, F.Cu at (173.5, 145.9)
- added J3: USB, Connector_PinHeader_2.54mm:PinHeader_1x04_P2.54mm_Vertical, F.Cu at (153.4, 145.9)
- added Q1: MMBT3904, Package_TO_SOT_SMD:SOT-23_Handsoldering, F.Cu at (180.2, 127.6)
- added Q2: MMBT3906, Package_TO_SOT_SMD:SOT-23_Handsoldering, F.Cu at (184.3, 127.6)
- added Q3: MMBT3904, Package_TO_SOT_SMD:SOT-23_Handsoldering, F.Cu at (171.9, 127.6)
- added Q4: MMBT3906, Package_TO_SOT_SMD:SOT-23_Handsoldering, F.Cu at (176.0, 127.6)
- added Q5: MMBT3904, Package_TO_SOT_SMD:SOT-23_Handsoldering, F.Cu at (180.2, 120.5)
- added Q6: MMBT3904, Package_TO_SOT_SMD:SOT-23_Handsoldering, F.Cu at (176.0, 120.5)
- added Q7: MMBT3904, Package_TO_SOT_SMD:SOT-23_Handsoldering, F.Cu at (184.3, 120.5)
- added Q8: MMBT3904, Package_TO_SOT_SMD:SOT-23_Handsoldering, F.Cu at (125.2, 142.4)
- added R1: 10k, Resistor_SMD:R_1206_3216Metric_Pad1.30x1.75mm_HandSolder, F.Cu at (182.1, 140.8)
- added R10: 10k, Resistor_SMD:R_1206_3216Metric_Pad1.30x1.75mm_HandSolder, F.Cu at (179.2, 114.9)
- added R11: 10k, Resistor_SMD:R_1206_3216Metric_Pad1.30x1.75mm_HandSolder, F.Cu at (181.7, 114.9)
- added R12: 10k, Resistor_SMD:R_1206_3216Metric_Pad1.30x1.75mm_HandSolder, F.Cu at (184.3, 114.9)
- added R13: 1k, Resistor_SMD:R_1206_3216Metric_Pad1.30x1.75mm_HandSolder, F.Cu at (119.2, 142.4)
- added R14: 0 (Current Limit / Volume Adj.), Resistor_SMD:R_1206_3216Metric_Pad1.30x1.75mm_HandSolder, F.Cu at (137.6, 142.4)
- added R2: 10k, Resistor_SMD:R_1206_3216Metric_Pad1.30x1.75mm_HandSolder, F.Cu at (171.9, 140.8)
- added R3: 10k, Resistor_SMD:R_1206_3216Metric_Pad1.30x1.75mm_HandSolder, F.Cu at (180.2, 135.8)
- added R4: 10k, Resistor_SMD:R_1206_3216Metric_Pad1.30x1.75mm_HandSolder, F.Cu at (182.7, 135.8)
- added R5: 10k, Resistor_SMD:R_1206_3216Metric_Pad1.30x1.75mm_HandSolder, F.Cu at (185.2, 135.8)
- added R6: 10k, Resistor_SMD:R_1206_3216Metric_Pad1.30x1.75mm_HandSolder, F.Cu at (170.9, 135.8)
- added R7: 10k, Resistor_SMD:R_1206_3216Metric_Pad1.30x1.75mm_HandSolder, F.Cu at (173.5, 135.8)
- added R8: 10k, Resistor_SMD:R_1206_3216Metric_Pad1.30x1.75mm_HandSolder, F.Cu at (176.0, 135.8)
- added R9: 10k, Resistor_SMD:R_1206_3216Metric_Pad1.30x1.75mm_HandSolder, F.Cu at (176.7, 114.9)
- added U1: ~, Footprints:YD-ESP32-S3 (ESP32-S3-DevKitC-1 USB-C Clone), F.Cu at (162.3, 108.6)
- added U2: ~, Footprints:3.2in SPI TFT Touch Module, F.Cu at (104.4, 51.4)
Routing:
- net +5V: track 0.00 -> 266.0 mm
- net MOSI: track 0.00 -> 166.9 mm
- net SCLK: track 0.00 -> 147.1 mm
- net MISO: track 0.00 -> 136.7 mm
- net +3V3: track 0.00 -> 99.6 mm, vias 0 -> 12
- net FOLLOWER_TRG: track 0.00 -> 88.8 mm
- net SD_CS: track 0.00 -> 77.0 mm
- net COINCIDENCE_TRG: track 0.00 -> 68.5 mm
- net MAIN_TRG: track 0.00 -> 61.9 mm
- net DISPLAY_CS: track 0.00 -> 53.9 mm
- net DISPLAY_RST: track 0.00 -> 50.3 mm
- net Net-(J3-Pin_3): track 0.00 -> 46.7 mm
- net DISPLAY_DC: track 0.00 -> 46.7 mm
- net Net-(J3-Pin_2): track 0.00 -> 46.1 mm
- net DISPLAY_LED: track 0.00 -> 38.6 mm
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- added copper zone on B.Cu, net GND
- added copper zone on F.Cu, net GND
Other:
- board outline added: 94.4 x 100 mm
- board text added: "H3"
- board text added: "H4"
- board text added: "H5"

Commit message: Finalizing Mainboard
Routing:
- net GND: track 10.1 -> 13.7 mm, vias 144 -> 146
- net Net-(J3-Pin_2): track 46.1 -> 46.8 mm
Other:
- board text added: "(BUZZER)"
- board text added: "(COINCIDENCE_TRG)"
- board text added: "(D_CS)"
- board text added: "(D_DC)"
- board text added: "(D_LED)"
- board text added: "(D_RST)"
- board text added: "(FOLLOWER_TRG)"
- board text added: "(MAIN_TRG)"
- board text added: "(MISO)"
- board text added: "(MOSI)"
- board text added: "(SCLK)"
- board text added: "(SD_CS)"
- board text added: "(T_CS)"
- board text added: "(T_IRQ)"
- board text added: "(USB D+)"
- board text added: "(USB D-)"
- board text added: "+"
- board text added: "+5V"
- board text added: "-"
- board text added: "3.2 inch 240x320 TFT SPI touchscreen + SD card reader Display driver: ILI9341 Touch driver: XPT2046"
- board text added: ": Geiger Counter Mainboard : 1.0 : 2024-01-08"
- board text added: "BUZZER"
- board text added: "DATA+"
- board text added: "DATA-"
- board text added: "FOLLOWER T."
- board text added: "GND"
- board text added: "MAIN TUBE"
- board text added: "PCB REV DAT"
- board text added: "PULSE"
- board text added: "SBM-20 Geiger Counter Geiger Counter Mainboard 1.0 Median Dispersion 2024 https://github.com/median-dispersion/SBM-20-Geiger-Counter"
- board text added: "USB"
